File: CAD/V1.2.0/CTRL & COMS.kicad_sch (KiCad schematic)
At the start: 73 parts, among them K2 U262-161N-4BVC11, K3 easyC-SMD, K4 JST-2pin-SMD, K5 HEADER_MALE_1X1_Inkplate, K6 HEADER_MALE_1X1_Inkplate, K7 HEADER_MALE_1X1_Inkplate, K8 HEADER_MALE_1X1_Inkplate, K9 HEADER_MALE_1X1_Inkplate, Q1 DNP, Q2 NPN, Q3 NPN, Q4 NMOS, Q5 PMOS, Q6 PMOS, Q7 SSM3J358R,LF, Q8 NPN, Q9 SSM3J358R,LF, SW1 YTSA007A0151803B, SW2 K2-1114SA-A4SW-06, U2 TPS3840PL27DBVR, U3 CH340C, U4 MCP73831T, U5 MC14093BDTR2G, U6 TPS7A2633DRVR

Commit message: Updating open source files.
Parts:
- R30: renamed from R26; value 10k -> 33k
- R31: renamed from R27; value 10k -> 33k
- renumbered C20 to C22, C22 to C23, C21 to C24, C23 to C25, C64 to C27, C27 to C28, C65 to C29, C66 to C30, C29 to C31, C24 to C32, C25 to C33, C30 to C34, C28 to C35, D11 to D8, D12 to D9, K2 to K1, K3 to K2, K5 to K3, K6 to K4, K7 to K5, K8 to K6, K9 to K7, K4 to K8, PAD3 to PAD1, PAD4 to PAD2, PAD6 to PAD3, PAD9 to PAD4, PAD1 to PAD6, PAD2 to PAD7, Q4 to Q2, Q5 to Q3, Q2 to Q4, Q3 to Q5, R23 to R22, R24 to R23, R25 to R24, R29 to R25, R33 to R26, R30 to R27, R31 to R28, R22 to R29, R35 to R32, R36 to R33, R37 to R34, R38 to R35, R34 to R36, R39 to R37, R28 to R38, R32 to R39, U3 to U2, U2 to U3, U5 to U4, U6 to U5, U4 to U6
Connections:
- net PWR-SW-A: now reaches R35.1, SW2.1, U4.8 (IN1C), U4.9 (IN2C)
- net RST-SW: now reaches R26.1, SW1.2
- net PWR-SW-B: now reaches C31.2, R37.1, SW2.2
- net CHRG-LED: now reaches D10.2 (K), U6.1 (STAT)
Other:
- note added: "BATTERY CONNECTOR"
- note added: "POWER LED SWITCH"
- note removed: "BATTERY CONNECTION"
- note removed: "If you need constant power supply and don't want to use ON/OFF SWITCH, use this resistor."
- note removed: "PWR SWITCH 3V3"
- note removed: "SHORT CIRCUIT RESISTOR FOR ON/OFF SWITCH"
- title: Soldered Inkplate 6PLUS -> Soldered Inkplate 6 FLICK
- moved on the sheet: C22, C23, C24, C25, C26, C27, C28, C29, C30, C31, C32, C33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
